Commit message: more stuff

File: hector_gazebo/hector_models/hector_sensors_description/urdf/generic_camera.urdf.xacro (robot description, xacro)
@@ -40,23 +40,20 @@
         <update_rate>30.0</update_rate>
           <camera name="head">
-          <horizontal_fov>1.3962634</horizontal_fov>
-          <image>
-            <width>800</width>
-            <height>800</height>
-            <format>R8G8B8</format>
-          </image>
-          <clip>
-            <near>0.02</near>
-            <far>300</far>
-          </clip>
-          <noise>
-            <type>gaussian</type>
-            <!-- Noise is sampled independently per pixel on each frame.
-                That pixel's noise value is added to each of its color
-                channels, which at that point lie in the range [0,1]. -->
-            <mean>0.0</mean>
-            <stddev>0.007</stddev>
-          </noise>
-        </camera>
+            <horizontal_fov>${hfov * M_PI / 180.0}</horizontal_fov>
+            <image>
+              <width>${res_x}</width>
+              <height>${res_y}</height>
+              <format>${image_format}</format>
+            </image>
+            <clip>
+              <near>0.02</near>
+              <far>300</far>
+            </clip>
+            <noise>
+              <type>gaussian</type>
+              <mean>0.0</mean>
+              <stddev>0.007</stddev>
+            </noise>
+          </camera>
         <!-- <camera>
           <horizontal_fov>${hfov * M_PI/180.0}</horizontal_fov>

File: hector_gazebo/hector_quadrotor/hector_quadrotor_description/urdf/quadrotor_base.urdf.xacro (robot description, xacro)
@@ -22,7 +22,7 @@
       </visual>
       <collision>
-        <origin xyz="0 0 0.0" rpy="0 0 0" /> <!-- Adjusted origin to center the box -->
+        <origin xyz="0 0 -0.05" rpy="0 0 0" /> <!-- Adjusted origin to center the box -->
         <geometry>
-          <box size="0.2 0.2 0.20" /> <!-- Width: 15 cm, Length: 20 cm, Height: 5 cm -->
+          <box size="0.15 0.2 0.05" /> <!-- Width: 15 cm, Length: 20 cm, Height: 5 cm -->
         </geometry>
       </collision>

File: hector_gazebo/hector_quadrotor/hector_quadrotor_description/urdf/quadrotor_with_cam.urdf.xacro (robot description, xacro)
@@ -8,5 +8,26 @@
     <!-- Forward facing camera -->
     <xacro:include filename="$(find hector_sensors_description)/urdf/generic_camera.urdf.xacro" />
-    <xacro:generic_camera name="front_cam" parent="base_link" ros_topic="camera/image" cam_info_topic="camera/camera_info" update_rate="10" res_x="320" res_y="240" image_format="R8G8B8" hfov="90">
+    <xacro:generic_camera
+        name="front_cam_wide"
+        parent="base_link"
+        ros_topic="camera/wide/image"
+        cam_info_topic="camera/wide/camera_info"
+        update_rate="10"
+        res_x="1920"
+        res_y="1080"
+        image_format="R8G8B8"
+        hfov="90">
+      <origin xyz="0.0 0.0 -0.06" rpy="0 0 0"/>
+    </xacro:generic_camera>
+    <xacro:generic_camera
+        name="front_cam_narrow"
+        parent="base_link"
+        ros_topic="camera/narrow/image"
+        cam_info_topic="camera/narrow/camera_info"
+        update_rate="10"
+        res_x="1920"
+        res_y="1080"
+        image_format="R8G8B8"
+        hfov="22.5">
       <origin xyz="0.0 0.0 -0.06" rpy="0 0 0"/>
     </xacro:generic_camera>
